File: bit/bit.kicad_sch (KiCad schematic)
At the start: 12 parts, among them J1 MID, J10 COL, J11 ROW, J2 COL, J3 ROW, J4 COL, J5 ROW, J6 COL, J7 ROW, J8 COL, J9 ROW

Commit message: Use SMD pads for the Bit
Parts:
- J10, J2, J3, J4, J5, J6, J7, J8, J9: footprint Connector_Wire:SolderWire-0.5sqmm_1x01_D0.9mm_OD2.1mm -> Connector_Wire:SolderWirePad_1x01_SMD_1x2mm
- J11: footprint Connector_Wire:SolderWire-0.5sqmm_1x01_D0.9mm_OD2.1mm -> Connector_Wire:SolderWirePad_1x01_SMD_5x10mm
Changed lines of the file:
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@@
       (effects (font (size 1.27 1.27)) (justify left))
     )
-    (property "Footprint" "Connector_Wire:SolderWire-0.5sqmm_1x01_D0.9mm_OD2.1mm" (id 2) (at 76.835 57.785 0)
+    (property "Footprint" "Connector_Wire:SolderWirePad_1x01_SMD_1x2mm" (id 2) (at 76.835 57.785 0)
       (effects (font (size 1.27 1.27)) hide)
     )
@@
       (effects (font (size 1.27 1.27)) (justify left))
     )
-    (property "Footprint" "Connector_Wire:SolderWire-0.5sqmm_1x01_D0.9mm_OD2.1mm" (id 2) (at 76.2 89.535 0)
+    (property "Footprint" "Connector_Wire:SolderWirePad_1x01_SMD_1x2mm" (id 2) (at 76.2 89.535 0)
       (effects (font (size 1.27 1.27)) hide)
     )
@@
       (effects (font (size 1.27 1.27)) (justify left))
     )
-    (property "Footprint" "Connector_Wire:SolderWire-0.5sqmm_1x01_D0.9mm_OD2.1mm" (id 2) (at 76.835 75.565 0)
+    (property "Footprint" "Connector_Wire:SolderWirePad_1x01_SMD_5x10mm" (id 2) (at 76.835 75.565 0)
       (effects (font (size 1.27 1.27)) hide)
     )
@@
       (effects (font (size 1.27 1.27)) (justify left))
     )
-    (property "Footprint" "Connector_Wire:SolderWire-0.5sqmm_1x01_D0.9mm_OD2.1mm" (id 2) (at 76.835 62.23 0)
+    (property "Footprint" "Connector_Wire:SolderWirePad_1x01_SMD_1x2mm" (id 2) (at 76.835 62.23 0)
       (effects (font (size 1.27 1.27)) hide)
     )
@@
       (effects (font (size 1.27 1.27)) (justify left))
     )
-    (property "Footprint" "Connector_Wire:SolderWire-0.5sqmm_1x01_D0.9mm_OD2.1mm" (id 2) (at 76.2 85.09 0)
+    (property "Footprint" "Connector_Wire:SolderWirePad_1x01_SMD_1x2mm" (id 2) (at 76.2 85.09 0)
       (effects (font (size 1.27 1.27)) hide)
     )
@@
       (effects (font (size 1.27 1.27)) (justify left))
     )
-    (property "Footprint" "Connector_Wire:SolderWire-0.5sqmm_1x01_D0.9mm_OD2.1mm" (id 2) (at 76.835 48.26 0)
+    (property "Footprint" "Connector_Wire:SolderWirePad_1x01_SMD_1x2mm" (id 2) (at 76.835 48.26 0)
       (effects (font (size 1.27 1.27)) hide)
     )
@@
       (effects (font (size 1.27 1.27)) (justify left))
     )
-    (property "Footprint" "Connector_Wire:SolderWire-0.5sqmm_1x01_D0.9mm_OD2.1mm" (id 2) (at 76.2 99.06 0)
+    (property "Footprint" "Connector_Wire:SolderWirePad_1x01_SMD_1x2mm" (id 2) (at 76.2 99.06 0)
       (effects (font (size 1.27 1.27)) hide)
     )
@@
       (effects (font (size 1.27 1.27)) (justify left))
     )
-    (property "Footprint" "Connector_Wire:SolderWire-0.5sqmm_1x01_D0.9mm_OD2.1mm" (id 2) (at 76.835 43.815 0)
+    (property "Footprint" "Connector_Wire:SolderWirePad_1x01_SMD_1x2mm" (id 2) (at 76.835 43.815 0)
       (effects (font (size 1.27 1.27)) hide)
     )
@@
       (effects (font (size 1.27 1.27)) (justify left))
     )
-    (property "Footprint" "Connector_Wire:SolderWire-0.5sqmm_1x01_D0.9mm_OD2.1mm" (id 2) (at 76.2 103.505 0)
+    (property "Footprint" "Connector_Wire:SolderWirePad_1x01_SMD_1x2mm" (id 2) (at 76.2 103.505 0)
       (effects (font (size 1.27 1.27)) hide)
     )
@@
       (effects (font (size 1.27 1.27)) (justify left))
     )
-    (property "Footprint" "Connector_Wire:SolderWire-0.5sqmm_1x01_D0.9mm_OD2.1mm" (id 2) (at 76.835 71.12 0)
+    (property "Footprint" "Connector_Wire:SolderWirePad_1x01_SMD_1x2mm" (id 2) (at 76.835 71.12 0)
       (effects (font (size 1.27 1.27)) hide)
     )
@@
     )
     (path "/bab44e03-7937-4a63-8b13-57fd1c0a3c29"
-      (reference "J2") (unit 1) (value "COL") (footprint "Connector_Wire:SolderWire-0.5sqmm_1x01_D0.9mm_OD2.1mm")
+      (reference "J2") (unit 1) (value "COL") (footprint "Connector_Wire:SolderWirePad_1x01_SMD_1x2mm")
     )
     (path "/5d1b7ea8-c279-4b06-9d74-610eff4d656b"
-      (reference "J3") (unit 1) (value "ROW") (footprint "Connector_Wire:SolderWire-0.5sqmm_1x01_D0.9mm_OD2.1mm")
+      (reference "J3") (unit 1) (value "ROW") (footprint "Connector_Wire:SolderWirePad_1x01_SMD_1x2mm")
     )
     (path "/5c06b5d7-eba1-486a-a175-16f13c32c88d"
-      (reference "J4") (unit 1) (value "COL") (footprint "Connector_Wire:SolderWire-0.5sqmm_1x01_D0.9mm_OD2.1mm")
+      (reference "J4") (unit 1) (value "COL") (footprint "Connector_Wire:SolderWirePad_1x01_SMD_1x2mm")
     )
     (path "/2bb13da1-2426-434d-851b-1fe455c62b35"
-      (reference "J5") (unit 1) (value "ROW") (footprint "Connector_Wire:SolderWire-0.5sqmm_1x01_D0.9mm_OD2.1mm")
+      (reference "J5") (unit 1) (value "ROW") (footprint "Connector_Wire:SolderWirePad_1x01_SMD_1x2mm")
     )
     (path "/9ec32fe4-8d35-4d14-9655-e88a0e49f933"
-      (reference "J6") (unit 1) (value "COL") (footprint "Connector_Wire:SolderWire-0.5sqmm_1x01_D0.9mm_OD2.1mm")
+      (reference "J6") (unit 1) (value "COL") (footprint "Connector_Wire:SolderWirePad_1x01_SMD_1x2mm")
     )
     (path "/d3d99902-dda4-450f-a50c-5db3792a60fa"
-      (reference "J7") (unit 1) (value "ROW") (footprint "Connector_Wire:SolderWire-0.5sqmm_1x01_D0.9mm_OD2.1mm")
+      (reference "J7") (unit 1) (value "ROW") (footprint "Connector_Wire:SolderWirePad_1x01_SMD_1x2mm")
     )
     (path "/2752f136-d3e0-42a8-9bd7-d900745ad735"
-      (reference "J8") (unit 1) (value "COL") (footprint "Connector_Wire:SolderWire-0.5sqmm_1x01_D0.9mm_OD2.1mm")
+      (reference "J8") (unit 1) (value "COL") (footprint "Connector_Wire:SolderWirePad_1x01_SMD_1x2mm")
     )
     (path "/587f9a17-6d42-41ae-9a6e-e9f800b385a7"
-      (reference "J9") (unit 1) (value "ROW") (footprint "Connector_Wire:SolderWire-0.5sqmm_1x01_D0.9mm_OD2.1mm")
+      (reference "J9") (unit 1) (value "ROW") (footprint "Connector_Wire:SolderWirePad_1x01_SMD_1x2mm")
     )
     (path "/dadd2fcc-55e3-4371-88bc-2a54e9ee3258"
-      (reference "J10") (unit 1) (value "COL") (footprint "Connector_Wire:SolderWire-0.5sqmm_1x01_D0.9mm_OD2.1mm")
+      (reference "J10") (unit 1) (value "COL") (footprint "Connector_Wire:SolderWirePad_1x01_SMD_1x2mm")
     )
     (path "/3678430b-c3b9-4dd4-b7e7-77462a7627ae"
-      (reference "J11") (unit 1) (value "ROW") (footprint "Connector_Wire:SolderWire-0.5sqmm_1x01_D0.9mm_OD2.1mm")
-    )
-  )
+      (reference "J11") (unit 1) (value "ROW") (footprint "Connector_Wire:SolderWirePad_1x01_SMD_5x10mm")
+    )
+  )
